File: GE_3T_Wantcom_motherboard.kicad_sch (KiCad schematic)
At the start: 29 parts, among them J1 Conn_01x03

Commit message: board with screws better placement, silkscreen issues
Parts:
- removed H1, H2, H3, H4: MountingHole, aaa_MyLib:screw head 440, symbol Mechanical:MountingHole
- added J2, J3, J4, J5: mounting screw, aaa_MyLib:screw head 440, symbol Connector:Conn_01x01_Socket
Connections:
- net GND: now also J2.1 (Pin_1), J3.1 (Pin_1), J4.1 (Pin_1), J5.1 (Pin_1)
